File: Dragon32.kicad_pcb (KiCad board)
At the start: 2 copper layers, 253 x 199.4 mm, 197 parts, among them IC1 HYB4116, IC10 2318, IC11 MC14053, IC12 MC6847, IC13 74LS273, IC14 74LS86, IC15 MC6883, IC16 74LS244, IC17 68A364, IC18 68A364, IC19 MC6809E, IC2 HYB4116, IC20 MC14529B, IC21 74LS123, IC22 74LS00, IC23 74LS74, IC24 74LS244, IC25 LM393, IC26 MC6821, IC27 74LS20, IC28 74LS393, IC29 74LS393, IC3 HYB4116, IC30 74LS32, IC31 74LS02, IC32 74LS390, IC33 74LS138, IC34 MC14050BCP, IC35 MC6821, IC4 HYB4116, IC5 HYB4116, IC6 HYB4116, IC7 HYB4116, IC8 HYB4116, IC9 LM1889N, SW1 RESET

Commit message: fix board dimensions
Parts:
- added C68: 0.1uF, Capacitor_THT:C_Disc_D3.0mm_W2.0mm_P2.50mm, F.Cu at (170.6, 158.0)
- added C69: 0.1uF, Capacitor_THT:C_Disc_D3.0mm_W2.0mm_P2.50mm, F.Cu at (170.6, 161.7)
- added JP11-12: printer/comms, Connector_PinHeader_2.54mm:PinHeader_1x03_P2.54mm_Vertical, F.Cu at (267.5, 122.6)
- added L3: 3.3uH, Inductor_THT:L_Axial_L7.0mm_D3.3mm_P10.16mm_Horizontal_Fastron_MICC, F.Cu at (96.3, 118.0)
- added L4: 3.3uH, Inductor_THT:L_Axial_L7.0mm_D3.3mm_P10.16mm_Horizontal_Fastron_MICC, F.Cu at (101.5, 70.6)
- moved L2 17.3 mm to (100.7, 104.5)
- moved L1 11.0 mm to (96.1, 70.7), turned to 90 degrees
- moved R17 10.2 mm to (133.3, 81.2), turned to 180 degrees
- moved R45 2.16 mm to (135.4, 164.2)
- moved R18 1.40 mm to (99.4, 74.0)
- moved PL5 0.85 mm to (86.8, 73.7)
- moved SW1 0.75 mm to (90.9, 35.7)
- moved PL4 0.37 mm to (86.8, 94.3)
Connections:
- C38 pad 2: PA1 -> PA0
- C39 pad 2: PA0 -> PA1
- IC35 pad 3: Net-(IC31-Pad8) -> Net-(IC35-Pad3)
- PL3 pad 6: unconnected-(PL3-Pad6) -> Net-(PL3-Pad6)
- PL5 pad 6: unconnected-(PL5-Pad6) -> Net-(PL5-Pad6)
Routing:
- net +12V: track 28.4 -> 216.6 mm, vias 0 -> 1
- net GND: track 1641.9 -> 1768.7 mm
- net +5V: track 1636.1 -> 1622.8 mm
Other:
- board size 253 x 199.4 mm -> 253 x 173.5 mm
- board text added: "parallel comms"
- board text added: "printer"

Commit message: add drill holes
Parts:
- moved PL2 3.14 mm to (86.7, 175.6)
Routing:
- net +5V: track 1622.8 -> 1615.0 mm
- net GND: track 1768.7 -> 1772.0 mm
Other:
- outline, holes or cut-outs redrawn
