File: Dragon32.kicad_pcb (KiCad board)
At the start: 2 copper layers, 253 x 173.5 mm, 207 parts, among them IC1 HYB4116, IC10 LM318, IC11 MC14053, IC12 MC6847, IC13 74LS273, IC14 74HC86, IC15 MC6883, IC16 74HC244, IC19 MC6809E, IC2 HYB4116, IC20 MC14529B, IC21 74HC123, IC22 74HC00, IC23 74HC74, IC24 74LS244, IC25 LM393, IC26 MC6821, IC27 74HC20, IC28 74HC393, IC29 74HC393, IC3 HYB4116, IC30 74HC32, IC31 74HC02, IC32 74HC390, IC33 74HC138, IC34 74HC245, IC35 MC6821, IC39 28C256, IC4 HYB4116, IC40 74HC08, IC5 HYB4116, IC6 HYB4116, IC7 HYB4116, IC8 HYB4116, IC9 LM1889N, SW1 RESET, SW2 SW_DIP_x02

Commit message: autoroute board
Parts:
- IC24: value 74LS244 -> 74HC244; footprint Package_DIP:DIP-20_W7.62mm -> Package_SO:SOIC-20W_7.5x12.8mm_P1.27mm
- TR1: value BC141 -> 2PD601; footprint Package_TO_SOT_THT:TO-92_Inline -> Package_TO_SOT_SMD:SOT-23
- TR2, TR3: value 2N2369 -> SMBT3904; footprint Package_TO_SOT_THT:TO-92_Inline -> Package_TO_SOT_SMD:SOT-23
- TR4: value BC212 -> SST3906; footprint Package_TO_SOT_THT:TO-92_Inline -> Package_TO_SOT_SMD:SOT-23
- moved C4 191.0 mm to (301.8, 82.8), turned to 0 degrees
- moved C48 184.1 mm to (94.9, 84.4), turned to 90 degrees
- moved R36 167.2 mm to (301.8, 80.1), turned to 180 degrees
- moved JP11-12 156.9 mm to (95.4, 179.1)
- moved D5 153.6 mm to (295.3, 82.8), turned to 180 degrees
- moved R15 152.7 mm to (154.7, 124.3), turned to -90 degrees
- moved D4 152.3 mm to (295.3, 85.5), turned to 180 degrees
- moved D6 147.8 mm to (295.3, 80.1), turned to 0 degrees
- moved R64 141.8 mm to (130.0, 153.5), turned to 0 degrees
- moved IC35 140.2 mm to (139.5, 144.3), turned to 90 degrees
- moved R56 137.9 mm to (116.6, 154.3)
- moved R62 136.6 mm to (130.0, 160.0), turned to 0 degrees
- moved R61 134.7 mm to (130.0, 157.9), turned to 0 degrees
- moved R60 132.9 mm to (130.0, 155.7), turned to 0 degrees
- moved R59 129.4 mm to (130.0, 166.5), turned to 0 degrees
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Routing:
- net GND: track 0.00 -> 1840.9 mm, vias 0 -> 47
- net +5V: track 0.00 -> 1641.8 mm, vias 0 -> 18
- net D2: track 0.00 -> 339.6 mm, vias 0 -> 7
- net D6: track 0.00 -> 336.1 mm, vias 0 -> 7
- net +12V: track 0.00 -> 326.7 mm, vias 0 -> 1
- net D4: track 0.00 -> 322.7 mm, vias 0 -> 4
- net D0: track 0.00 -> 322.2 mm, vias 0 -> 7
- net D1: track 0.00 -> 312.9 mm, vias 0 -> 7
- net D3: track 0.00 -> 306.5 mm, vias 0 -> 4
- net D7: track 0.00 -> 305.0 mm, vias 0 -> 6
- net D5: track 0.00 -> 297.8 mm, vias 0 -> 6
- net Net-(C4-Pad1): track 0.00 -> 293.2 mm, vias 0 -> 2
- net E: track 0.00 -> 278.2 mm, vias 0 -> 3
- net A1: track 0.00 -> 256.6 mm, vias 0 -> 4
- net DO0: track 0.00 -> 253.5 mm, vias 0 -> 3
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Other:
- board text added: "Revision ex"
- board text removed: "Revision 1.2"

Commit message: complete wiring
Routing:
- net Net-(IC31-Pad8): track 1.27 -> 173.9 mm, vias 0 -> 10
- net Net-(IC33-Pad5): track 0.00 -> 171.2 mm, vias 0 -> 16
- net Net-(IC31-Pad4): track 0.00 -> 155.4 mm, vias 0 -> 18
- net Net-(IC31-Pad1): track 0.00 -> 147.8 mm, vias 0 -> 18
- net Z7: track 40.6 -> 171.0 mm, vias 1 -> 10
- net GND: track 1840.9 -> 1963.4 mm, vias 47 -> 56
- net Net-(IC35-Pad12): track 0.00 -> 113.5 mm, vias 0 -> 7
- net Net-(IC35-Pad3): track 0.00 -> 76.5 mm, vias 0 -> 5
- net RAM VBB: track 134.2 -> 186.2 mm, vias 0 -> 7
- net RAM VCC: track 114.9 -> 154.2 mm, vias 2 -> 4
- net RAM VDD: track 143.3 -> 182.4 mm, vias 0 -> 3
- net STROBE: track 195.1 -> 206.5 mm
- net +5V: track 1641.8 -> 1650.7 mm
- net ~{E18}: track 110.8 -> 105.5 mm
- net A6: track 140.0 -> 145.0 mm
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