File: mpu.kicad_sch (KiCad schematic)
At the start: 14 parts, among them IC19 MC6809E, SW1 RESET

Commit message: convert to smd
Parts:
- C22: footprint Capacitor_THT:CP_Radial_D6.3mm_P2.50mm -> Capacitor_SMD:CP_Elec_6.3x3.9
- C23: footprint Capacitor_THT:CP_Radial_D5.0mm_P2.50mm -> Capacitor_SMD:CP_Elec_5x3
- C4: footprint Capacitor_THT:C_Disc_D3.0mm_W2.0mm_P2.50mm -> Capacitor_SMD:C_0805_2012Metric
- D4, D5, D6: footprint Diode_THT:D_DO-35_SOD27_P7.62mm_Horizontal -> Diode_SMD:D_0805_2012Metric
- R13, R14, R15, R36, R40, R41: footprint Resistor_THT:R_Axial_DIN0207_L6.3mm_D2.5mm_P10.16mm_Horizontal -> Resistor_SMD:R_0805_2012Metric
Changed lines of the file:
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@@
     (property "Reference" "D6" (id 0) (at 96.1644 91.694 0))
     (property "Value" "1N914" (id 1) (at 93.853 91.694 0))
-    (property "Footprint" "Diode_THT:D_DO-35_SOD27_P7.62mm_Horizontal" (id 2) (at 86.233 91.694 0)
+    (property "Footprint" "Diode_SMD:D_0805_2012Metric" (id 2) (at 86.233 91.694 0)
       (effects (font (size 1.27 1.27)) hide)
     )
@@
     (property "Reference" "C22" (id 0) (at 173.8693 52.197 90))
     (property "Value" "100uF" (id 1) (at 173.8693 54.737 90))
-    (property "Footprint" "Capacitor_THT:CP_Radial_D6.3mm_P2.50mm" (id 2) (at 173.863 58.674 0)
+    (property "Footprint" "Capacitor_SMD:CP_Elec_6.3x3.9" (id 2) (at 173.863 58.674 0)
       (effects (font (size 1.27 1.27)) hide)
     )
@@
       (effects (font (size 1.27 1.27)) (justify left))
     )
-    (property "Footprint" "Resistor_THT:R_Axial_DIN0207_L6.3mm_D2.5mm_P10.16mm_Horizontal" (id 2) (at 137.668 104.394 0)
+    (property "Footprint" "Resistor_SMD:R_0805_2012Metric" (id 2) (at 137.668 104.394 0)
       (effects (font (size 1.27 1.27)) hide)
     )
@@
       (effects (font (size 1.27 1.27)) (justify left))
     )
-    (property "Footprint" "Resistor_THT:R_Axial_DIN0207_L6.3mm_D2.5mm_P10.16mm_Horizontal" (id 2) (at 121.412 81.534 90)
+    (property "Footprint" "Resistor_SMD:R_0805_2012Metric" (id 2) (at 121.412 81.534 90)
       (effects (font (size 1.27 1.27)) hide)
     )
@@
       (effects (font (size 1.27 1.27)) (justify left))
     )
-    (property "Footprint" "Resistor_THT:R_Axial_DIN0207_L6.3mm_D2.5mm_P10.16mm_Horizontal" (id 2) (at 100.33 91.694 90)
+    (property "Footprint" "Resistor_SMD:R_0805_2012Metric" (id 2) (at 100.33 91.694 90)
       (effects (font (size 1.27 1.27)) hide)
     )
@@
     (property "Reference" "D5" (id 0) (at 75.0316 91.694 0))
     (property "Value" "1N914" (id 1) (at 77.343 91.694 0))
-    (property "Footprint" "Diode_THT:D_DO-35_SOD27_P7.62mm_Horizontal" (id 2) (at 84.963 91.694 0)
+    (property "Footprint" "Diode_SMD:D_0805_2012Metric" (id 2) (at 84.963 91.694 0)
       (effects (font (size 1.27 1.27)) hide)
     )
@@
     (property "Reference" "D4" (id 0) (at 86.0044 101.854 0))
     (property "Value" "1N914" (id 1) (at 83.693 101.854 0))
-    (property "Footprint" "Diode_THT:D_DO-35_SOD27_P7.62mm_Horizontal" (id 2) (at 76.073 101.854 0)
+    (property "Footprint" "Diode_SMD:D_0805_2012Metric" (id 2) (at 76.073 101.854 0)
       (effects (font (size 1.27 1.27)) hide)
     )
@@
       (effects (font (size 1.27 1.27)) (justify left))
     )
-    (property "Footprint" "Resistor_THT:R_Axial_DIN0207_L6.3mm_D2.5mm_P10.16mm_Horizontal" (id 2) (at 144.653 98.425 0)
+    (property "Footprint" "Resistor_SMD:R_0805_2012Metric" (id 2) (at 144.653 98.425 0)
       (effects (font (size 1.27 1.27)) hide)
     )
@@
       (effects (font (size 1.27 1.27)) (justify left))
     )
-    (property "Footprint" "Capacitor_THT:C_Disc_D3.0mm_W2.0mm_P2.50mm" (id 2) (at 90.678 101.854 0)
+    (property "Footprint" "Capacitor_SMD:C_0805_2012Metric" (id 2) (at 90.678 101.854 0)
       (effects (font (size 1.27 1.27)) hide)
     )
@@
       (effects (font (size 1.27 1.27)) (justify left))
     )
-    (property "Footprint" "Resistor_THT:R_Axial_DIN0207_L6.3mm_D2.5mm_P10.16mm_Horizontal" (id 2) (at 151.511 98.425 0)
+    (property "Footprint" "Resistor_SMD:R_0805_2012Metric" (id 2) (at 151.511 98.425 0)
       (effects (font (size 1.27 1.27)) hide)
     )
@@
       (effects (font (size 1.27 1.27)) (justify left))
     )
-    (property "Footprint" "Resistor_THT:R_Axial_DIN0207_L6.3mm_D2.5mm_P10.16mm_Horizontal" (id 2) (at 137.668 98.425 0)
+    (property "Footprint" "Resistor_SMD:R_0805_2012Metric" (id 2) (at 137.668 98.425 0)
       (effects (font (size 1.27 1.27)) hide)
     )
@@
       (effects (font (size 1.27 1.27)) (justify left))
     )
-    (property "Footprint" "Capacitor_THT:CP_Radial_D5.0mm_P2.50mm" (id 2) (at 123.19 92.964 0)
-      (effects (font (size 1.27 1.27)) hide)
-    )
+    (property "Footprint" "Capacitor_SMD:CP_Elec_5x3" (id 2) (at 123.19 92.964 0)
+      (effects (font (size 1.27 1.27)) hide)
+    )
