File: mpu.kicad_sch (KiCad schematic)
At the start: 14 parts, among them IC19 MC6809E, SW1 RESET

Commit message: update bom references
Parts:
- IC19: Mouser (none) -> 517-4840-6000-CP
Changed lines of the file:
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@@
+			)
+		)
+		(property "Mouser" "517-4840-6000-CP"
+			(at 168.148 94.234 0)
+			(effects
+				(font
+					(size 1.27 1.27)
+				)
+				(hide yes)
 			)
 		)

Commit message: fix parallel strobe inverter bypass
Other:
- company: (none) -> Dragon Data
Changed lines of the file:
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@@
 		(date "2023-06-03")
 		(rev "2.1")
+		(company "Dragon Data")
+		(comment 1 "Reproduced and Modified by Julian Brown")
 	)
 	(junction
