File: rom.kicad_sch (KiCad schematic)
At the start: 5 parts, among them IC39 28C256, IC40 74HC08, SW2 SW_DIP_x02

Commit message: swap new and gate over to a single circuit chip
Parts:
- removed IC40: 74HC08, Package_SO:SOIC-14_3.9x8.7mm_P1.27mm, symbol 74xx:74LS08
- added IC40: 74HC1G08, Package_SO:TSOP-5_1.65x3.05mm_P0.95mm, symbol vdg:74HC1G08
Connections:
- net +5V: now also IC40.5 (Vcc)
- net GND: now also IC40.3 (Gnd)
- net ~{E17}: now also IC40.1 (IN_B)
- net ~{E18}: now also IC40.2 (IN_A)
- net at IC39.22 (~{OE}): now also IC40.4 (OUT_Y)
- no-connect marks 9 -> 0
