File: rom.kicad_sch (KiCad schematic)
At the start: 2 parts, among them IC17 68A364, IC18 68A364

Commit message: update part numbers
Parts:
- IC17, IC18: Note (none) -> donor only
Changed lines of the file:
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@@
+      (effects (font (size 1.27 1.27)) hide)
+    )
+    (property "DigiKey" "" (id 4) (at 116.205 90.551 0)
+      (effects (font (size 1.27 1.27)) hide)
+    )
+    (property "Note" "donor only" (id 5) (at 116.205 90.551 0)
       (effects (font (size 1.27 1.27)) hide)
     )
@@
       (effects (font (size 1.27 1.27)) hide)
     )
+    (property "DigiKey" "" (id 4) (at 153.289 90.551 0)
+      (effects (font (size 1.27 1.27)) hide)
+    )
+    (property "Note" "donor only" (id 5) (at 153.289 90.551 0)
+      (effects (font (size 1.27 1.27)) hide)
+    )
