File: rom.kicad_sch (KiCad schematic)
At the start: 2 parts, among them IC17 68A364, IC18 68A364

Commit message: update bom references
Parts:
- IC17, IC18: Mouser (none) -> 517-4824-6000-CP
Changed lines of the file:
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@@
+			)
+		)
+		(property "Mouser" "517-4824-6000-CP"
+			(at 116.205 90.551 0)
+			(effects
+				(font
+					(size 1.27 1.27)
+				)
+				(hide yes)
 			)
 		)
@@
 			(at 153.289 90.551 0)
 			(effects
+				(font
+					(size 1.27 1.27)
+				)
+				(hide yes)
+			)
+		)
+		(property "Mouser" "517-4824-6000-CP"
+			(at 153.289 90.551 0)
+			(effects

Commit message: fix parallel strobe inverter bypass
Other:
- company: (none) -> Dragon Data
Changed lines of the file:
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@@
 		(date "2023-06-03")
 		(rev "2.1")
+		(company "Dragon Data")
+		(comment 1 "Reproduced and Modified by Julian Brown")
 	)
 	(global_label "A8"
