File: pia1.kicad_sch (KiCad schematic)
At the start: 33 parts, among them IC20 MC14529B, IC24 74LS244, IC25 LM393, IC26 MC6821

Commit message: validate component values
Parts:
- C1, C43, C45: value 0.1uF -> 0.01uF; footprint Capacitor_THT:C_Disc_D3.0mm_W2.0mm_P2.50mm -> Capacitor_THT:C_Disc_D4.3mm_W1.9mm_P5.00mm
- C30, C31, C32, C33: value 0.02uF -> 0.022uF; footprint Capacitor_THT:C_Disc_D3.0mm_W2.0mm_P2.50mm -> Capacitor_THT:C_Disc_D5.0mm_W2.5mm_P5.00mm
- C38, C39, C68, C69: footprint Capacitor_THT:C_Disc_D3.0mm_W2.0mm_P2.50mm -> Capacitor_THT:C_Disc_D4.3mm_W1.9mm_P5.00mm
Changed lines of the file:
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@@
       (effects (font (size 1.27 1.27)) (justify right))
     )
-    (property "Value" "0.1uF" (id 1) (at 260.604 68.0655 0)
-      (effects (font (size 1.27 1.27)) (justify right))
-    )
-    (property "Footprint" "Capacitor_THT:C_Disc_D3.0mm_W2.0mm_P2.50mm" (id 2) (at 257.429 66.802 0)
+    (property "Value" "0.01uF" (id 1) (at 260.604 68.0655 0)
+      (effects (font (size 1.27 1.27)) (justify right))
+    )
+    (property "Footprint" "Capacitor_THT:C_Disc_D4.3mm_W1.9mm_P5.00mm" (id 2) (at 257.429 66.802 0)
       (effects (font (size 1.27 1.27)) hide)
     )
@@
       (effects (font (size 1.27 1.27)) (justify right))
     )
-    (property "Footprint" "Capacitor_THT:C_Disc_D3.0mm_W2.0mm_P2.50mm" (id 2) (at 113.538 70.866 0)
+    (property "Footprint" "Capacitor_THT:C_Disc_D4.3mm_W1.9mm_P5.00mm" (id 2) (at 113.538 70.866 0)
       (effects (font (size 1.27 1.27)) hide)
     )
@@
       (effects (font (size 1.27 1.27)) (justify right))
     )
-    (property "Footprint" "Capacitor_THT:C_Disc_D3.0mm_W2.0mm_P2.50mm" (id 2) (at 84.328 70.866 0)
+    (property "Footprint" "Capacitor_THT:C_Disc_D4.3mm_W1.9mm_P5.00mm" (id 2) (at 84.328 70.866 0)
       (effects (font (size 1.27 1.27)) hide)
     )
@@
     (in_bom yes) (on_board yes) (fields_autoplaced)
     (property "Reference" "C45" (id 0) (at 53.4606 40.64 90))
-    (property "Value" "0.1uF" (id 1) (at 53.4606 43.18 90))
-    (property "Footprint" "Capacitor_THT:C_Disc_D3.0mm_W2.0mm_P2.50mm" (id 2) (at 53.467 47.498 0)
+    (property "Value" "0.01uF" (id 1) (at 53.4606 43.18 90))
+    (property "Footprint" "Capacitor_THT:C_Disc_D4.3mm_W1.9mm_P5.00mm" (id 2) (at 53.467 47.498 0)
       (effects (font (size 1.27 1.27)) hide)
     )
@@
       (effects (font (size 1.27 1.27)) (justify right))
     )
-    (property "Value" "0.02uF" (id 1) (at 222.504 44.8245 0)
-      (effects (font (size 1.27 1.27)) (justify right))
-    )
-    (property "Footprint" "Capacitor_THT:C_Disc_D3.0mm_W2.0mm_P2.50mm" (id 2) (at 219.329 43.561 0)
+    (property "Value" "0.022uF" (id 1) (at 222.504 44.8245 0)
+      (effects (font (size 1.27 1.27)) (justify right))
+    )
+    (property "Footprint" "Capacitor_THT:C_Disc_D5.0mm_W2.5mm_P5.00mm" (id 2) (at 219.329 43.561 0)
       (effects (font (size 1.27 1.27)) hide)
     )
@@
       (effects (font (size 1.27 1.27)) (justify right))
     )
-    (property "Footprint" "Capacitor_THT:C_Disc_D3.0mm_W2.0mm_P2.50mm" (id 2) (at 103.378 70.866 0)
+    (property "Footprint" "Capacitor_THT:C_Disc_D4.3mm_W1.9mm_P5.00mm" (id 2) (at 103.378 70.866 0)
       (effects (font (size 1.27 1.27)) hide)
     )
@@
     (in_bom yes) (on_board yes) (fields_autoplaced)
     (property "Reference" "C43" (id 0) (at 95.7516 133.223 90))
-    (property "Value" "0.1uF" (id 1) (at 95.7516 135.763 90))
-    (property "Footprint" "Capacitor_THT:C_Disc_D3.0mm_W2.0mm_P2.50mm" (id 2) (at 95.758 140.208 0)
+    (property "Value" "0.01uF" (id 1) (at 95.7516 135.763 90))
+    (property "Footprint" "Capacitor_THT:C_Disc_D4.3mm_W1.9mm_P5.00mm" (id 2) (at 95.758 140.208 0)
       (effects (font (size 1.27 1.27)) hide)
     )
@@
       (effects (font (size 1.27 1.27)) (justify right))
     )
-    (property "Value" "0.02uF" (id 1) (at 210.185 91.4335 0)
-      (effects (font (size 1.27 1.27)) (justify right))
-    )
-    (property "Footprint" "Capacitor_THT:C_Disc_D3.0mm_W2.0mm_P2.50mm" (id 2) (at 207.01 90.17 0)
+    (property "Value" "0.022uF" (id 1) (at 210.185 91.4335 0)
+      (effects (font (size 1.27 1.27)) (justify right))
+    )
+    (property "Footprint" "Capacitor_THT:C_Disc_D5.0mm_W2.5mm_P5.00mm" (id 2) (at 207.01 90.17 0)
       (effects (font (size 1.27 1.27)) hide)
     )
@@
       (effects (font (size 1.27 1.27)) hide)
     )
-    (pin "1")
-    (pin "2")
-    (pin "3")
     (pin "5")
     (pin "6")
     (pin "7")
-    (pin "4")
-    (pin "8")
   )
   (symbol (lib_id "power:GND") (at 197.866 153.162 0) (unit 1)
@@
       (effects (font (size 1.27 1.27)) (justify right))
     )
-    (property "Value" "0.02uF" (id 1) (at 210.185 44.8245 0)
-      (effects (font (size 1.27 1.27)) (justify right))
-    )
-    (property "Footprint" "Capacitor_THT:C_Disc_D3.0mm_W2.0mm_P2.50mm" (id 2) (at 207.01 43.561 0)
+    (property "Value" "0.022uF" (id 1) (at 210.185 44.8245 0)
+      (effects (font (size 1.27 1.27)) (justify right))
+    )
+    (property "Footprint" "Capacitor_THT:C_Disc_D5.0mm_W2.5mm_P5.00mm" (id 2) (at 207.01 43.561 0)
       (effects (font (size 1.27 1.27)) hide)
     )
@@
       (effects (font (size 1.27 1.27)) (justify right))
     )
-    (property "Footprint" "Capacitor_THT:C_Disc_D3.0mm_W2.0mm_P2.50mm" (id 2) (at 94.488 70.866 0)
+    (property "Footprint" "Capacitor_THT:C_Disc_D4.3mm_W1.9mm_P5.00mm" (id 2) (at 94.488 70.866 0)
       (effects (font (size 1.27 1.27)) hide)
     )
@@
       (effects (font (size 1.27 1.27)) (justify right))
     )
-    (property "Value" "0.02uF" (id 1) (at 222.504 91.4335 0)
-      (effects (font (size 1.27 1.27)) (justify right))
-    )
-    (property "Footprint" "Capacitor_THT:C_Disc_D3.0mm_W2.0mm_P2.50mm" (id 2) (at 219.329 90.17 0)
-      (effects (font (size 1.27 1.27)) hide)
-    )
+    (property "Value" "0.022uF" (id 1) (at 222.504 91.4335 0)
+      (effects (font (size 1.27 1.27)) (justify right))
+    )
+    (property "Footprint" "Capacitor_THT:C_Disc_D5.0mm_W2.5mm_P5.00mm" (id 2) (at 219.329 90.17 0)
+      (effects (font (size 1.27 1.27)) hide)
+    )

Commit message: cross-reference items to suppliers
Parts:
- IC24: value 74LS244 -> 74LS244N; DigiKey (none) -> 296-1653-5-ND
- IC25: value LM393 -> LM393P; DigiKey (none) -> 296-1398-5-ND
Changed lines of the file:
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@@
       (effects (font (size 1.27 1.27)) (justify left))
     )
-    (property "Value" "74LS244" (id 1) (at 102.4764 143.51 0)
+    (property "Value" "74LS244N" (id 1) (at 102.4764 143.51 0)
       (effects (font (size 1.27 1.27)) (justify left))
     )
@@
     )
     (property "Datasheet" "http://www.ti.com/lit/ds/symlink/sn74ls244.pdf" (id 3) (at 100.457 161.671 0)
+      (effects (font (size 1.27 1.27)) hide)
+    )
+    (property "DigiKey" "296-1653-5-ND" (id 4) (at 100.457 161.671 0)
       (effects (font (size 1.27 1.27)) hide)
     )
@@
     (in_bom yes) (on_board yes)
     (property "Reference" "IC25" (id 0) (at 258.064 147.447 0))
-    (property "Value" "LM393" (id 1) (at 256.413 154.305 0))
+    (property "Value" "LM393P" (id 1) (at 256.413 154.305 0))
     (property "Footprint" "Package_DIP:DIP-8_W7.62mm" (id 2) (at 258.064 154.432 0)
       (effects (font (size 1.27 1.27)) hide)
@@
       (effects (font (size 1.27 1.27)) hide)
     )
+    (property "DigiKey" "296-1398-5-ND" (id 4) (at 258.064 154.432 0)
+      (effects (font (size 1.27 1.27)) hide)
+    )

Commit message: update part numbers
Parts:
- C1, C43, C45: DigiKey (none) -> BC2662CT-ND
- C30, C31, C32, C33: value 0.022uF -> 22nF; DigiKey (none) -> BC2677CT-ND
- C38, C39, C68, C69: DigiKey (none) -> BC1101CT-ND
- D8, D9: DigiKey (none) -> 1N914FS-ND
- PL2: DigiKey (none) -> CHR20G-ND; Note (none) -> or 1195-1707-ND with latches
Changed lines of the file:
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@@
       (effects (font (size 1.27 1.27)) hide)
     )
-    (property "Datasheet" "~" (id 3) (at 197.866 144.78 90)
+    (property "Datasheet" "http://www.vishay.com/docs/85622/1n914.pdf" (id 3) (at 197.866 144.78 90)
+      (effects (font (size 1.27 1.27)) hide)
+    )
+    (property "DigiKey" "1N914FS-ND" (id 4) (at 197.866 144.78 0)
       (effects (font (size 1.27 1.27)) hide)
     )
@@
       (effects (font (size 1.27 1.27)) hide)
     )
-    (property "Datasheet" "~" (id 3) (at 257.429 66.802 0)
+    (property "Datasheet" "https://www.vishay.com/docs/45171/kseries.pdf" (id 3) (at 257.429 66.802 0)
+      (effects (font (size 1.27 1.27)) hide)
+    )
+    (property "DigiKey" "BC2662CT-ND" (id 4) (at 257.429 66.802 0)
       (effects (font (size 1.27 1.27)) hide)
     )
@@
       (effects (font (size 1.27 1.27)) hide)
     )
-    (property "Datasheet" "~" (id 3) (at 113.538 70.866 0)
+    (property "Datasheet" "https://www.vishay.com/docs/45171/kseries.pdf" (id 3) (at 113.538 70.866 0)
+      (effects (font (size 1.27 1.27)) hide)
+    )
+    (property "DigiKey" "BC1101CT-ND" (id 4) (at 113.538 70.866 0)
       (effects (font (size 1.27 1.27)) hide)
     )
@@
       (effects (font (size 1.27 1.27)) hide)
     )
-    (property "Datasheet" "http://www.mouser.com/ds/2/18/40_c091_abd_e-75918.pdf" (id 3) (at 230.378 27.686 0)
+    (property "Datasheet" "https://www.dem-uk.com/deltron-components/Data/Product_Downloads/deltron-671-0501-5-way-din-socket-data.pdf" (id 3) (at 230.378 27.686 0)
       (effects (font (size 1.27 1.27)) hide)
     )
@@
       (effects (font (size 1.27 1.27)) hide)
     )
-    (property "Datasheet" "~" (id 3) (at 84.328 70.866 0)
+    (property "Datasheet" "https://www.vishay.com/docs/45171/kseries.pdf" (id 3) (at 84.328 70.866 0)
+      (effects (font (size 1.27 1.27)) hide)
+    )
+    (property "DigiKey" "BC1101CT-ND" (id 4) (at 84.328 70.866 0)
       (effects (font (size 1.27 1.27)) hide)
     )
@@
       (effects (font (size 1.27 1.27)) hide)
     )
-    (property "Datasheet" "http://www.mouser.com/ds/2/18/40_c091_abd_e-75918.pdf" (id 3) (at 230.378 74.676 0)
+    (property "Datasheet" "https://www.dem-uk.com/deltron-components/Data/Product_Downloads/deltron-671-0501-5-way-din-socket-data.pdf" (id 3) (at 230.378 74.676 0)
       (effects (font (size 1.27 1.27)) hide)
     )
@@
       (effects (font (size 1.27 1.27)) hide)
     )
-    (property "Datasheet" "~" (id 3) (at 53.467 47.498 0)
+    (property "Datasheet" "https://www.vishay.com/docs/45171/kseries.pdf" (id 3) (at 53.467 47.498 0)
+      (effects (font (size 1.27 1.27)) hide)
+    )
+    (property "DigiKey" "BC2662CT-ND" (id 4) (at 53.467 47.498 0)
       (effects (font (size 1.27 1.27)) hide)
     )
@@
       (effects (font (size 1.27 1.27)) hide)
     )
-    (property "Datasheet" "~" (id 3) (at 197.866 150.495 90)
+    (property "Datasheet" "http://www.vishay.com/docs/85622/1n914.pdf" (id 3) (at 197.866 150.495 90)
+      (effects (font (size 1.27 1.27)) hide)
+    )
+    (property "DigiKey" "1N914FS-ND" (id 4) (at 197.866 150.495 0)
       (effects (font (size 1.27 1.27)) hide)
     )
@@
       (effects (font (size 1.27 1.27)) (justify right))
     )
-    (property "Value" "0.022uF" (id 1) (at 222.504 44.8245 0)
+    (property "Value" "22nF" (id 1) (at 222.504 44.8245 0)
       (effects (font (size 1.27 1.27)) (justify right))
     )
@@
       (effects (font (size 1.27 1.27)) hide)
     )
-    (property "Datasheet" "~" (id 3) (at 219.329 43.561 0)
+    (property "Datasheet" "https://www.vishay.com/docs/45171/kseries.pdf" (id 3) (at 219.329 43.561 0)
+      (effects (font (size 1.27 1.27)) hide)
+    )
+    (property "DigiKey" "BC2677CT-ND" (id 4) (at 219.329 43.561 0)
       (effects (font (size 1.27 1.27)) hide)
     )
@@
       (effects (font (size 1.27 1.27)) hide)
     )
-    (property "Datasheet" "~" (id 3) (at 103.378 70.866 0)
+    (property "Datasheet" "https://www.vishay.com/docs/45171/kseries.pdf" (id 3) (at 103.378 70.866 0)
+      (effects (font (size 1.27 1.27)) hide)
+    )
+    (property "DigiKey" "BC1101CT-ND" (id 4) (at 103.378 70.866 0)
       (effects (font (size 1.27 1.27)) hide)
     )
@@
       (effects (font (size 1.27 1.27)) hide)
     )
-    (property "Datasheet" "~" (id 3) (at 95.758 140.208 0)
+    (property "Datasheet" "https://www.vishay.com/docs/45171/kseries.pdf" (id 3) (at 95.758 140.208 0)
+      (effects (font (size 1.27 1.27)) hide)
+    )
+    (property "DigiKey" "BC2662CT-ND" (id 4) (at 95.758 140.208 0)
       (effects (font (size 1.27 1.27)) hide)
     )
@@
       (effects (font (size 1.27 1.27)) hide)
     )
-    (property "Datasheet" "~" (id 3) (at 149.606 157.226 0)
+    (property "Datasheet" "https://media.digikey.com/pdf/Data%20Sheets/CW%20Industries%20PDFs/CWN-300%20Ordering.pdf" (id 3) (at 149.606 157.226 0)
+      (effects (font (size 1.27 1.27)) hide)
+    )
+    (property "DigiKey" "CHR20G-ND" (id 4) (at 149.606 157.226 0)
+      (effects (font (size 1.27 1.27)) hide)
+    )
+    (property "Note" "or 1195-1707-ND with latches" (id 5) (at 149.606 157.226 0)
       (effects (font (size 1.27 1.27)) hide)
     )
@@
       (effects (font (size 1.27 1.27)) (justify right))
     )
-    (property "Value" "0.022uF" (id 1) (at 210.185 91.4335 0)
+    (property "Value" "22nF" (id 1) (at 210.185 91.4335 0)
       (effects (font (size 1.27 1.27)) (justify right))
     )
@@
       (effects (font (size 1.27 1.27)) hide)
     )
-    (property "Datasheet" "~" (id 3) (at 207.01 90.17 0)
+    (property "Datasheet" "https://www.vishay.com/docs/45171/kseries.pdf" (id 3) (at 207.01 90.17 0)
+      (effects (font (size 1.27 1.27)) hide)
+    )
+    (property "DigiKey" "BC2677CT-ND" (id 4) (at 207.01 90.17 0)
       (effects (font (size 1.27 1.27)) hide)
     )
@@
       (effects (font (size 1.27 1.27)) (justify right))
     )
-    (property "Value" "0.022uF" (id 1) (at 210.185 44.8245 0)
+    (property "Value" "22nF" (id 1) (at 210.185 44.8245 0)
       (effects (font (size 1.27 1.27)) (justify right))
     )
@@
       (effects (font (size 1.27 1.27)) hide)
     )
-    (property "Datasheet" "~" (id 3) (at 207.01 43.561 0)
+    (property "Datasheet" "https://www.vishay.com/docs/45171/kseries.pdf" (id 3) (at 207.01 43.561 0)
+      (effects (font (size 1.27 1.27)) hide)
+    )
+    (property "DigiKey" "BC2677CT-ND" (id 4) (at 207.01 43.561 0)
       (effects (font (size 1.27 1.27)) hide)
     )
@@
       (effects (font (size 1.27 1.27)) hide)
     )
-    (property "Datasheet" "~" (id 3) (at 94.488 70.866 0)
+    (property "Datasheet" "https://www.vishay.com/docs/45171/kseries.pdf" (id 3) (at 94.488 70.866 0)
+      (effects (font (size 1.27 1.27)) hide)
+    )
+    (property "DigiKey" "BC1101CT-ND" (id 4) (at 94.488 70.866 0)
       (effects (font (size 1.27 1.27)) hide)
     )
@@
       (effects (font (size 1.27 1.27)) (justify right))
     )
-    (property "Value" "0.022uF" (id 1) (at 222.504 91.4335 0)
+    (property "Value" "22nF" (id 1) (at 222.504 91.4335 0)
       (effects (font (size 1.27 1.27)) (justify right))
     )
@@
       (effects (font (size 1.27 1.27)) hide)
     )
-    (property "Datasheet" "~" (id 3) (at 219.329 90.17 0)
-      (effects (font (size 1.27 1.27)) hide)
-    )
+    (property "Datasheet" "https://www.vishay.com/docs/45171/kseries.pdf" (id 3) (at 219.329 90.17 0)
+      (effects (font (size 1.27 1.27)) hide)
+    )
+    (property "DigiKey" "BC2677CT-ND" (id 4) (at 219.329 90.17 0)
+      (effects (font (size 1.27 1.27)) hide)
+    )

Commit message: resolve part numbers
Parts:
- IC20: DigiKey (none) -> CD4529BCN-ND; Note (none) -> obsolete, use donor
- IC26: DigiKey (none) -> 2156-MC6821CS-2156-ND; Note (none) -> donor is preferable
- L1, L2, L3, L4: DigiKey (none) -> 495-5561-1-ND
- PL1: DigiKey (none) -> 952-2521-ND
- PL3, PL5: Note (none) -> RS Components
- R1: DigiKey (none) -> CF14JT100RCT-ND
- R30, R31: DigiKey (none) -> CF14JT4K70CT-ND
- R42, R43, R55: DigiKey (none) -> CF14JT10K0CT-ND
- R53: DigiKey (none) -> CF14JT10M0CT-ND
- R54: DigiKey (none) -> CF14JT1K00CT-ND
Changed lines of the file:
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@@
+      (effects (font (size 1.27 1.27)) hide)
+    )
+    (property "DigiKey" "2156-MC6821CS-2156-ND" (id 4) (at 58.928 85.344 0)
+      (effects (font (size 1.27 1.27)) hide)
+    )
+    (property "Note" "donor is preferable" (id 5) (at 58.928 85.344 0)
       (effects (font (size 1.27 1.27)) hide)
     )
@@
       (effects (font (size 1.27 1.27)) hide)
     )
+    (property "DigiKey" "CF14JT4K70CT-ND" (id 4) (at 190.119 144.653 0)
+      (effects (font (size 1.27 1.27)) hide)
+    )
     (pin "1")
     (pin "2")
@@
       (effects (font (size 1.27 1.27)) hide)
     )
+    (property "DigiKey" "CF14JT10K0CT-ND" (id 4) (at 246.888 145.034 0)
+      (effects (font (size 1.27 1.27)) hide)
+    )
     (pin "1")
     (pin "2")
@@
     )
     (property "Datasheet" "~" (id 3) (at 190.119 150.495 0)
+      (effects (font (size 1.27 1.27)) hide)
+    )
+    (property "DigiKey" "CF14JT4K70CT-ND" (id 4) (at 190.119 150.495 0)
       (effects (font (size 1.27 1.27)) hide)
     )
@@
     )
     (property "Datasheet" "https://www.dem-uk.com/deltron-components/Data/Product_Downloads/deltron-671-0501-5-way-din-socket-data.pdf" (id 3) (at 230.378 27.686 0)
+      (effects (font (size 1.27 1.27)) hide)
+    )
+    (property "Note" "RS Components" (id 4) (at 230.378 27.686 0)
       (effects (font (size 1.27 1.27)) hide)
     )
@@
       (effects (font (size 1.27 1.27)) hide)
     )
+    (property "DigiKey" "CF14JT10M0CT-ND" (id 4) (at 262.001 145.034 0)
+      (effects (font (size 1.27 1.27)) hide)
+    )
     (pin "1")
     (pin "2")
@@
     )
     (property "Datasheet" "https://www.dem-uk.com/deltron-components/Data/Product_Downloads/deltron-671-0501-5-way-din-socket-data.pdf" (id 3) (at 230.378 74.676 0)
+      (effects (font (size 1.27 1.27)) hide)
+    )
+    (property "Note" "RS Components" (id 4) (at 230.378 74.676 0)
       (effects (font (size 1.27 1.27)) hide)
     )
@@
     )
     (property "Datasheet" "" (id 3) (at 227.33 137.414 0)
+      (effects (font (size 1.27 1.27)) hide)
+    )
+    (property "DigiKey" "CD4529BCN-ND" (id 4) (at 227.33 137.414 0)
+      (effects (font (size 1.27 1.27)) hide)
+    )
+    (property "Note" "obsolete, use donor" (id 5) (at 227.33 137.414 0)
       (effects (font (size 1.27 1.27)) hide)
     )
@@
       (effects (font (size 1.27 1.27)) hide)
     )
+    (property "DigiKey" "CF14JT10K0CT-ND" (id 4) (at 167.894 174.244 0)
+      (effects (font (size 1.27 1.27)) hide)
+    )
     (pin "1")
     (pin "2")
@@
       (effects (font (size 1.27 1.27)) hide)
     )
+    (property "DigiKey" "CF14JT100RCT-ND" (id 4) (at 261.366 61.976 0)
+      (effects (font (size 1.27 1.27)) hide)
+    )
     (pin "1")
     (pin "2")
@@
     )
     (property "Datasheet" "~" (id 3) (at 240.538 72.136 0)
+      (effects (font (size 1.27 1.27)) hide)
+    )
+    (property "DigiKey" "495-5561-1-ND" (id 4) (at 240.538 72.136 0)
       (effects (font (size 1.27 1.27)) hide)
     )
@@
       (effects (font (size 1.27 1.27)) hide)
     )
+    (pin "1")
+    (pin "2")
+    (pin "3")
     (pin "5")
     (pin "6")
     (pin "7")
+    (pin "4")
+    (pin "8")
   )
   (symbol (lib_id "power:GND") (at 197.866 153.162 0) (unit 1)
@@
       (effects (font (size 1.27 1.27)) hide)
     )
+    (property "DigiKey" "CF14JT10K0CT-ND" (id 4) (at 157.988 174.244 0)
+      (effects (font (size 1.27 1.27)) hide)
+    )
     (pin "1")
     (pin "2")
@@
     )
     (property "Datasheet" "~" (id 3) (at 265.684 142.494 0)
+      (effects (font (size 1.27 1.27)) hide)
+    )
+    (property "DigiKey" "CF14JT1K00CT-ND" (id 4) (at 265.684 142.494 0)
       (effects (font (size 1.27 1.27)) hide)
     )
@@
       (effects (font (size 1.27 1.27)) hide)
     )
+    (property "DigiKey" "495-5561-1-ND" (id 4) (at 230.378 37.846 0)
+      (effects (font (size 1.27 1.27)) hide)
+    )
     (pin "1")
     (pin "2")
@@
     )
     (property "Datasheet" "~" (id 3) (at 148.209 41.656 0)
+      (effects (font (size 1.27 1.27)) hide)
+    )
+    (property "DigiKey" "952-2521-ND" (id 4) (at 148.209 41.656 0)
       (effects (font (size 1.27 1.27)) hide)
     )
@@
       (effects (font (size 1.27 1.27)) hide)
     )
+    (property "DigiKey" "495-5561-1-ND" (id 4) (at 230.378 84.836 0)
+      (effects (font (size 1.27 1.27)) hide)
+    )
     (pin "1")
     (pin "2")
@@
       (effects (font (size 1.27 1.27)) hide)
     )
+    (property "DigiKey" "495-5561-1-ND" (id 4) (at 240.538 25.146 0)
+      (effects (font (size 1.27 1.27)) hide)
+    )
