File: pia1.kicad_sch (KiCad schematic)
At the start: 33 parts, among them IC20 MC14529B, IC24 74LS244N, IC25 LM393P, IC26 MC6821

Commit message: update board for revision 2.2
Parts:
- added PL9: CoCo Keyboard, Connector_PinHeader_2.54mm:PinHeader_1x16_P2.54mm_Vertical, symbol Connector:Conn_01x16_Male
- PL1: value Conn_01x16_Male -> Dragon Keyboard
Connections:
- net GND: now also PL9.3 (Pin_3)
- net PA0: now also PL9.6 (Pin_6)
- net PA1: now also PL9.7 (Pin_7)
- net PA2: now also PL9.1 (Pin_1)
- net PA3: now also PL9.2 (Pin_2)
- net PA4: now also PL9.4 (Pin_4)
- net PA5: now also PL9.5 (Pin_5)
- net PA6: now also PL9.8 (Pin_8)
- net PB0: now also PL9.9 (Pin_9)
- net PB1: now also PL9.10 (Pin_10)
- net PB2: now also PL9.11 (Pin_11)
- net PB3: now also PL9.12 (Pin_12)
- net PB4: now also PL9.13 (Pin_13)
- net PB5: now also PL9.14 (Pin_14)
- net PB6: now also PL9.15 (Pin_15)
- net PB7: now also PL9.16 (Pin_16)

Commit message: update bom references
Parts:
- C38, C39, C68, C69: DigiKey BC1101CT-ND -> BC2662CT-ND
- IC26: DigiKey 2156-MC6821CS-2156-ND -> (none); Mouser (none) -> 517-4840-6000-CP
- PL3, PL5: DigiKey (none) -> CP-7060-ND
- PL9: DigiKey 952-2521-ND -> (none); Mouser (none) -> 538-22-28-8161
Changed lines of the file:
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@@
 			)
 		)
-		(property "DigiKey" "2156-MC6821CS-2156-ND"
+		(property "DigiKey" ""
 			(at 58.928 85.344 0)
 			(effects
@@
 			)
 		)
+		(property "Mouser" "517-4840-6000-CP"
+			(at 58.928 85.344 0)
+			(effects
+				(font
+					(size 1.27 1.27)
+				)
+				(hide yes)
+			)
+		)
 		(pin "1"
 		)
@@
 			)
 		)
-		(property "DigiKey" "BC1101CT-ND"
+		(property "DigiKey" "BC2662CT-ND"
 			(at 113.538 70.866 0)
 			(effects
@@
 			)
 		)
+		(property "DigiKey" "CP-7060-ND"
+			(at 230.378 27.686 0)
+			(effects
+				(font
+					(size 1.27 1.27)
+				)
+				(hide yes)
+			)
+		)
 		(pin "1"
 		)
@@
 			)
 		)
-		(property "DigiKey" "BC1101CT-ND"
+		(property "DigiKey" "BC2662CT-ND"
 			(at 84.328 70.866 0)
 			(effects
@@
 			)
 		)
+		(property "DigiKey" "CP-7060-ND"
+			(at 230.378 74.676 0)
+			(effects
+				(font
+					(size 1.27 1.27)
+				)
+				(hide yes)
+			)
+		)
 		(pin "1"
 		)
@@
 			)
 		)
-		(property "DigiKey" "BC1101CT-ND"
+		(property "DigiKey" "BC2662CT-ND"
 			(at 103.378 70.866 0)
 			(effects
@@
 			)
 		)
-		(property "DigiKey" "BC1101CT-ND"
+		(property "DigiKey" "BC2662CT-ND"
 			(at 94.488 70.866 0)
 			(effects
@@
 			)
 		)
-		(property "DigiKey" "952-2521-ND"
+		(property "DigiKey" ""
+			(at 173.482 41.148 0)
+			(effects
+				(font
+					(size 1.27 1.27)
+				)
+				(hide yes)
+			)
+		)
+		(property "Mouser" "538-22-28-8161"
 			(at 173.482 41.148 0)
 			(effects

Commit message: fix parallel strobe inverter bypass
Other:
- company: (none) -> Dragon Data
Changed lines of the file:
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@@
 		(date "2023-06-03")
 		(rev "2.1")
+		(company "Dragon Data")
+		(comment 1 "Reproduced and Modified by Julian Brown")
 	)
 	(junction
