File: vdg.kicad_sch (KiCad schematic)
At the start: 3 parts, among them IC12 MC6847, IC13 74LS273N

Commit message: update board for revision 2.2
Connections:
- net GD4: now reaches IC12.7 (D4), IC13.12 (Q4)
- net GD5: now reaches IC12.8 (D5), IC13.15 (Q5)
- net GD6: now reaches IC12.2 (D6), IC12.32 (INV), IC13.16 (Q6)
- net GD7: now reaches IC12.34 (~{A}/S), IC12.40 (D7), IC13.19 (Q7)
- net GD0: now reaches IC12.3 (D0), IC13.2 (Q0)
- net GD1: now reaches IC12.4 (D1), IC13.5 (Q1)
- net GD2: now reaches IC12.5 (D2), IC13.6 (Q2)
- net GD3: now reaches IC12.6 (D3), IC13.9 (Q3)

Commit message: update bom references
Parts:
- IC12: Mouser (none) -> 517-4840-6000-CP
Changed lines of the file:
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@@
+			)
+		)
+		(property "Mouser" "517-4840-6000-CP"
+			(at 162.56 101.092 0)
+			(effects
+				(font
+					(size 1.27 1.27)
+				)
+				(hide yes)
 			)
 		)

Commit message: fix parallel strobe inverter bypass
Other:
- company: (none) -> Dragon Data
Changed lines of the file:
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@@
 		(date "2023-06-03")
 		(rev "2.1")
+		(company "Dragon Data")
+		(comment 1 "Reproduced and Modified by Julian Brown")
 	)
 	(junction
